File: MagicWheelchair-Mega-Shield/MW-Mega-Shield.brd (EAGLE design)
At the start: 87.3 x 58.4 mm, 20 parts

Commit message: Update PCB, add PNG version
Parts:
- moved TOUCH_DISABLE 53.9 mm to (16.5, 31.8), turned to 90 degrees
- moved R3 48.2 mm to (16.1, 38.1), turned to 180 degrees
- moved R2 20.1 mm to (26.7, 49.5)
- moved R1 17.3 mm to (39.4, 49.5)
Connections:
- net TOUCH_DISABLE: now also B1.12; no longer B1.5
Routing:
- net TOUCH_DISABLE: track 18.5 -> 46.6 mm
- net UNDER_DATA: track 26.7 -> 5.50 mm
- net N$2: track 7.82 -> 29.1 mm
- net FIRE_DATA: track 24.1 -> 5.50 mm
- net N$1: track 7.30 -> 24.9 mm
- net VIN: track 89.2 -> 97.6 mm
- net INPUT_OPT: track 17.2 -> 16.5 mm
