File: MagicWheelchair-Mega-Shield/old/MW-Mega-Shield.sch (EAGLE design)
At the start: 21 parts

Commit message: Merge shields into one
Parts:
- B1: value ARDUINO_MEGA_R3FULL -> ARDUINO_MEGA_R3-SIMPLE; device SparkFun-Boards:ARDUINO_MEGA_R3FULL -> SparkFun-Boards:ARDUINO_MEGA_R3-SIMPLE
Connections:
- net GND: now also B1.GND@0, B1.GND@1, B1.GND@4, J1.1, J3.1; no longer J1.3, J3.3
- net N$1: now also B1.13; no longer B1.10
- net N$2: now also B1.5; no longer B1.6
- net N$4: now also B1.2; no longer B1.15(RX3)
- net N$5: now also B1.21(SCL); no longer B1.19(RX1)
- net RIGHT_5V: now also J3.3; no longer J3.1
- net TOUCH_DISABLE: no longer B1.14(TX3)
- net VIN: now also B1.VIN, J1.3; no longer J1.1
Other:
- moved on the sheet: R2, R3, R5
Changed lines of the file:
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@@
 </classes>
 <parts>
+<part name="B1" library="SparkFun-Boards" library_urn="urn:adsk.eagle:library:509" deviceset="ARDUINO_MEGA_R3-SIMPLE" device=""/>
 <part name="R1" library="rcl" library_urn="urn:adsk.eagle:library:334" deviceset="R-US_" device="R0603" package3d_urn="urn:adsk.eagle:package:23555/2" value="30kOhm"/>
 <part name="R2" library="rcl" library_urn="urn:adsk.eagle:library:334" deviceset="R-US_" device="R0603" package3d_urn="urn:adsk.eagle:package:23555/2" value="30kOhm"/>
@@
 <part name="R3" library="rcl" library_urn="urn:adsk.eagle:library:334" deviceset="R-US_" device="R0603" package3d_urn="urn:adsk.eagle:package:23555/2" value="30kOhm"/>
 <part name="R5" library="rcl" library_urn="urn:adsk.eagle:library:334" deviceset="R-US_" device="R0603" package3d_urn="urn:adsk.eagle:package:23555/2" value="30kOhm"/>
-<part name="B1" library="SparkFun-Boards" deviceset="ARDUINO_MEGA_R3" device="FULL"/>
 </parts>
 <sheets>
@@
 </plain>
 <instances>
+<instance part="B1" gate="G$1" x="66.04" y="63.5"/>
 <instance part="R1" gate="G$1" x="93.98" y="114.3" rot="MR0"/>
-<instance part="R2" gate="G$1" x="91.44" y="88.9" rot="MR0"/>
+<instance part="R2" gate="G$1" x="22.86" y="27.94"/>
 <instance part="C1" gate="G$1" x="-17.78" y="142.24"/>
 <instance part="5V-IN" gate="G$1" x="-35.56" y="147.32"/>
@@
 <instance part="DUMMY_STAND1" gate="G$1" x="-50.8" y="63.5"/>
 <instance part="DUMMY_STAND3" gate="G$1" x="-50.8" y="48.26"/>
-<instance part="R3" gate="G$1" x="91.44" y="66.04" rot="MR0"/>
-<instance part="R5" gate="G$1" x="91.44" y="55.88" rot="MR0"/>
-<instance part="B1" gate="B1" x="60.96" y="68.58"/>
+<instance part="R3" gate="G$1" x="22.86" y="60.96"/>
+<instance part="R5" gate="G$1" x="91.44" y="93.98" rot="MR0"/>
 </instances>
 <busses>
@@
 </segment>
 <segment>
+<pinref part="B1" gate="G$1" pin="GND@0"/>
+<wire x1="48.26" y1="22.86" x2="35.56" y2="22.86" width="0.1524" layer="91"/>
+<label x="30.48" y="22.86" size="1.778" layer="95"/>
+</segment>
+<segment>
+<pinref part="B1" gate="G$1" pin="GND@1"/>
+<wire x1="48.26" y1="20.32" x2="35.56" y2="20.32" width="0.1524" layer="91"/>
+<label x="30.48" y="20.32" size="1.778" layer="95"/>
+</segment>
+<segment>
+<pinref part="B1" gate="G$1" pin="GND@4"/>
+<wire x1="48.26" y1="12.7" x2="35.56" y2="12.7" width="0.1524" layer="91"/>
+<label x="30.48" y="12.7" size="1.778" layer="95"/>
+</segment>
+<segment>
 <pinref part="S1" gate="1" pin="S"/>
 <wire x1="149.86" y1="25.4" x2="149.86" y2="15.24" width="0.1524" layer="91"/>
@@
 </segment>
 <segment>
+<pinref part="J1" gate="J$1" pin="1"/>
+<wire x1="142.24" y1="124.46" x2="160.02" y2="124.46" width="0.1524" layer="91"/>
+<label x="165.1" y="124.46" size="1.778" layer="95"/>
+</segment>
+<segment>
 <pinref part="J2" gate="J$1" pin="1"/>
 <wire x1="142.24" y1="109.22" x2="160.02" y2="109.22" width="0.1524" layer="91"/>
 <label x="165.1" y="109.22" size="1.778" layer="95"/>
+</segment>
+<segment>
+<pinref part="J3" gate="J$1" pin="1"/>
+<wire x1="142.24" y1="88.9" x2="160.02" y2="88.9" width="0.1524" layer="91"/>
+<label x="165.1" y="88.9" size="1.778" layer="95"/>
 </segment>
 <segment>
@@
 <junction x="68.58" y="132.08"/>
 </segment>
-<segment>
-<pinref part="J1" gate="J$1" pin="3"/>
-<wire x1="142.24" y1="129.54" x2="160.02" y2="129.54" width="0.1524" layer="91"/>
-<label x="165.1" y="129.54" size="1.778" layer="95"/>
-</segment>
-<segment>
-<pinref part="J3" gate="J$1" pin="3"/>
-<wire x1="142.24" y1="93.98" x2="160.02" y2="93.98" width="0.1524" layer="91"/>
-<label x="165.1" y="93.98" size="1.778" layer="95"/>
-</segment>
 </net>
 <net name="VIN" class="0">
+<segment>
+<pinref part="B1" gate="G$1" pin="VIN"/>
+<wire x1="48.26" y1="114.3" x2="38.1" y2="114.3" width="0.1524" layer="91"/>
+<label x="33.02" y="114.3" size="1.778" layer="95"/>
+</segment>
 <segment>
 <pinref part="C1" gate="G$1" pin="+"/>
@@
 </segment>
 <segment>
+<pinref part="J1" gate="J$1" pin="3"/>
+<wire x1="142.24" y1="129.54" x2="160.02" y2="129.54" width="0.1524" layer="91"/>
+<label x="165.1" y="129.54" size="1.778" layer="95"/>
+</segment>
+<segment>
 <pinref part="J2" gate="J$1" pin="3"/>
 <wire x1="142.24" y1="114.3" x2="160.02" y2="114.3" width="0.1524" layer="91"/>
 <label x="165.1" y="114.3" size="1.778" layer="95"/>
 </segment>
-<segment>
-<pinref part="J1" gate="J$1" pin="1"/>
-<wire x1="142.24" y1="124.46" x2="160.02" y2="124.46" width="0.1524" layer="91"/>
-<label x="165.1" y="124.46" size="1.778" layer="95"/>
-</segment>
 </net>
 <net name="TOUCH_DISABLE" class="0">
@@
 <label x="96.52" y="27.94" size="1.778" layer="95"/>
 </segment>
-<segment>
-<pinref part="B1" gate="B1" pin="14(TX3)"/>
-<wire x1="76.2" y1="68.58" x2="81.28" y2="68.58" width="0.1524" layer="91"/>
-<wire x1="81.28" y1="68.58" x2="81.28" y2="73.66" width="0.1524" layer="91"/>
-<wire x1="81.28" y1="73.66" x2="91.44" y2="73.66" width="0.1524" layer="91"/>
-<label x="93.98" y="73.66" size="1.778" layer="95"/>
-</segment>
 </net>
 <net name="N$3" class="0">
@@
 <segment>
 <pinref part="R2" gate="G$1" pin="1"/>
-<wire x1="96.52" y1="88.9" x2="111.76" y2="88.9" width="0.1524" layer="91"/>
-<label x="124.46" y="88.9" size="1.778" layer="95" rot="MR0"/>
+<wire x1="17.78" y1="27.94" x2="2.54" y2="27.94" width="0.1524" layer="91"/>
+<label x="-10.16" y="27.94" size="1.778" layer="95"/>
 </segment>
 </net>
@@
 <segment>
 <pinref part="R3" gate="G$1" pin="1"/>
-<wire x1="96.52" y1="66.04" x2="124.46" y2="66.04" width="0.1524" layer="91"/>
-<label x="124.46" y="66.04" size="1.778" layer="95" rot="MR0"/>
+<wire x1="17.78" y1="60.96" x2="-10.16" y2="60.96" width="0.1524" layer="91"/>
+<label x="-10.16" y="60.96" size="1.778" layer="95"/>
 </segment>
 </net>
@@
 <wire x1="142.24" y1="78.74" x2="160.02" y2="78.74" width="0.1524" layer="91"/>
 <label x="165.1" y="78.74" size="1.778" layer="95"/>
+</segment>
+<segment>
+<pinref part="J3" gate="J$1" pin="3"/>
+<wire x1="142.24" y1="93.98" x2="160.02" y2="93.98" width="0.1524" layer="91"/>
+<label x="165.1" y="93.98" size="1.778" layer="95"/>
 </segment>
 <segment>
@@
 <junction x="68.58" y="147.32"/>
 </segment>
-<segment>
-<pinref part="J3" gate="J$1" pin="1"/>
-<wire x1="142.24" y1="88.9" x2="160.02" y2="88.9" width="0.1524" layer="91"/>
-<label x="165.1" y="88.9" size="1.778" layer="95"/>
-</segment>
 </net>
 <net name="UNDER_RIGHT_DATA" class="0">
@@
 <segment>
 <pinref part="R5" gate="G$1" pin="1"/>
-<wire x1="96.52" y1="55.88" x2="124.46" y2="55.88" width="0.1524" layer="91"/>
-<label x="124.46" y="55.88" size="1.778" layer="95" rot="MR0"/>
+<wire x1="96.52" y1="93.98" x2="124.46" y2="93.98" width="0.1524" layer="91"/>
+<label x="124.46" y="93.98" size="1.778" layer="95" rot="MR0"/>
 </segment>
 </net>
@@
 <segment>
 <pinref part="R1" gate="G$1" pin="2"/>
+<pinref part="B1" gate="G$1" pin="13"/>
 <wire x1="88.9" y1="114.3" x2="83.82" y2="114.3" width="0.1524" layer="91"/>
-<wire x1="83.82" y1="114.3" x2="83.82" y2="101.6" width="0.1524" layer="91"/>
-<pinref part="B1" gate="B1" pin="10"/>
-<wire x1="83.82" y1="101.6" x2="76.2" y2="101.6" width="0.1524" layer="91"/>
 </segment>
 </net>
@@
 <segment>
 <pinref part="R5" gate="G$1" pin="2"/>
-<pinref part="B1" gate="B1" pin="19(RX1)"/>
-<wire x1="86.36" y1="55.88" x2="76.2" y2="55.88" width="0.1524" layer="91"/>
+<pinref part="B1" gate="G$1" pin="21(SCL)"/>
+<wire x1="86.36" y1="93.98" x2="83.82" y2="93.98" width="0.1524" layer="91"/>
 </segment>
 </net>
@@
 <segment>
 <pinref part="R2" gate="G$1" pin="2"/>
-<pinref part="B1" gate="B1" pin="6"/>
-<wire x1="86.36" y1="88.9" x2="76.2" y2="88.9" width="0.1524" layer="91"/>
+<wire x1="27.94" y1="27.94" x2="38.1" y2="27.94" width="0.1524" layer="91"/>
+<wire x1="38.1" y1="27.94" x2="38.1" y2="43.18" width="0.1524" layer="91"/>
+<pinref part="B1" gate="G$1" pin="5"/>
+<wire x1="38.1" y1="43.18" x2="48.26" y2="43.18" width="0.1524" layer="91"/>
 </segment>
 </net>
 <net name="N$4" class="0">
 <segment>
-<pinref part="B1" gate="B1" pin="15(RX3)"/>
 <pinref part="R3" gate="G$1" pin="2"/>
-<wire x1="76.2" y1="66.04" x2="86.36" y2="66.04" width="0.1524" layer="91"/>
-</segment>
-</net>
+<wire x1="27.94" y1="60.96" x2="35.56" y2="60.96" width="0.1524" layer="91"/>
+<wire x1="35.56" y1="60.96" x2="35.56" y2="50.8" width="0.1524" layer="91"/>
+<pinref part="B1" gate="G$1" pin="2"/>
+<wire x1="35.56" y1="50.8" x2="48.26" y2="50.8" width="0.1524" layer="91"/>
+</segment>
+</net>
